File: pcb/aek67.kicad_pcb (KiCad board)
At the start: 2 copper layers, 304.8 x 100.4 mm, 154 parts, among them J1 AVR-ISP-6, K1 K_GRV, K10 K_9, K11 K_0, K12 K_MINUS, K13 K_EQUAL, K14 K_BACKSPACE, K15 K_PAGE_UP, K16 K_TAB, K17 K_Q, K18 K_W, K19 K_E, K2 K_1, K20 K_R, K21 K_T, K22 K_Y, K23 K_U, K24 K_I, K25 K_O, K26 K_P, K27 K_LBRC, K28 K_RBRC, K29 K_BSLSH, K3 K_2, K30 K_PAGE_DN, K31 K_CAPS_LOCK, K32 K_A, K33 K_S, K34 K_D, K35 K_F, K36 K_G, K37 K_H, K38 K_J, K39 K_K, K4 K_3, K40 K_L, K41 K_SEMIC, K42 K_QUOTE, K43 K_ENTER, K44 K_INSERT, K45 K_LSHIFT, K46 K_Z, K47 K_X, K48 K_C, K49 K_V, K5 K_4, K50 K_B, K51 K_N, K52 K_M, K53 K_COMMA, K54 K_DOT, K55 K_SLASH, K56 K_RSHIFT, K57 K_UP, K58 K_DELETE, K59 K_LCTRL, K6 K_5, K60 K_LAPP, K61 K_LALT, K62 K_SPC, K63 K_RALT, K64 K_RAPP, K65 K_LEFT, K66 K_DOWN, K67 K_RIGHT, K7 K_6, K8 K_7, K9 K_8, SW1 SW_PUSH, U1 ATmega32U4-AU, U2 PRTR5V0U2X, X1 XTAL_GND

Commit message: row3
Routing:
- net row3: track 0.00 -> 381.3 mm, vias 0 -> 14
Changed lines of the file:
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@@
     (thickness 1.6)
     (drawings 14)
-    (tracks 770)
+    (tracks 829)
     (zones 0)
     (modules 154)
@@
   (segment (start 93.89375 25.6625) (end 96.04375 27.8125) (width 0.25) (layer B.Cu) (net 11))
   (segment (start 89.8125 25.6625) (end 93.89375 25.6625) (width 0.25) (layer B.Cu) (net 11))
+  (via (at 51.5 95.75) (size 0.8) (drill 0.4) (layers F.Cu B.Cu) (net 12))
+  (segment (start 50.8 95.05) (end 51.5 95.75) (width 0.25) (layer B.Cu) (net 12))
+  (segment (start 50.8 88.16875) (end 50.8 95.05) (width 0.25) (layer B.Cu) (net 12))
+  (via (at 80.5 95.75) (size 0.8) (drill 0.4) (layers F.Cu B.Cu) (net 12))
+  (segment (start 51.5 95.75) (end 80.5 95.75) (width 0.25) (layer F.Cu) (net 12))
+  (segment (start 81.75625 94.49375) (end 81.75625 88.16875) (width 0.25) (layer B.Cu) (net 12))
+  (segment (start 80.5 95.75) (end 81.75625 94.49375) (width 0.25) (layer B.Cu) (net 12))
+  (via (at 99.5 95.75) (size 0.8) (drill 0.4) (layers F.Cu B.Cu) (net 12))
+  (segment (start 80.5 95.75) (end 99.5 95.75) (width 0.25) (layer F.Cu) (net 12))
+  (segment (start 100.80625 94.44375) (end 100.80625 88.16875) (width 0.25) (layer B.Cu) (net 12))
+  (segment (start 99.5 95.75) (end 100.80625 94.44375) (width 0.25) (layer B.Cu) (net 12))
+  (via (at 118.5 95.75) (size 0.8) (drill 0.4) (layers F.Cu B.Cu) (net 12))
+  (segment (start 99.5 95.75) (end 118.5 95.75) (width 0.25) (layer F.Cu) (net 12))
+  (segment (start 119.85625 94.39375) (end 119.85625 88.16875) (width 0.25) (layer B.Cu) (net 12))
+  (segment (start 118.5 95.75) (end 119.85625 94.39375) (width 0.25) (layer B.Cu) (net 12))
+  (via (at 137.5 95.75) (size 0.8) (drill 0.4) (layers F.Cu B.Cu) (net 12))
+  (segment (start 118.5 95.75) (end 137.5 95.75) (width 0.25) (layer F.Cu) (net 12))
+  (segment (start 138.90625 94.34375) (end 138.90625 88.16875) (width 0.25) (layer B.Cu) (net 12))
+  (segment (start 137.5 95.75) (end 138.90625 94.34375) (width 0.25) (layer B.Cu) (net 12))
+  (via (at 156.5 95.75) (size 0.8) (drill 0.4) (layers F.Cu B.Cu) (net 12))
+  (segment (start 137.5 95.75) (end 156.5 95.75) (width 0.25) (layer F.Cu) (net 12))
+  (segment (start 157.95625 94.29375) (end 157.95625 88.16875) (width 0.25) (layer B.Cu) (net 12))
+  (segment (start 156.5 95.75) (end 157.95625 94.29375) (width 0.25) (layer B.Cu) (net 12))
+  (via (at 175.75 95.75) (size 0.8) (drill 0.4) (layers F.Cu B.Cu) (net 12))
+  (segment (start 156.5 95.75) (end 175.75 95.75) (width 0.25) (layer F.Cu) (net 12))
+  (segment (start 177.00625 94.49375) (end 177.00625 88.16875) (width 0.25) (layer B.Cu) (net 12))
+  (segment (start 175.75 95.75) (end 177.00625 94.49375) (width 0.25) (layer B.Cu) (net 12))
+  (via (at 194.75 95.75) (size 0.8) (drill 0.4) (layers F.Cu B.Cu) (net 12))
+  (segment (start 175.75 95.75) (end 194.75 95.75) (width 0.25) (layer F.Cu) (net 12))
+  (segment (start 196.05625 94.44375) (end 196.05625 88.16875) (width 0.25) (layer B.Cu) (net 12))
+  (segment (start 194.75 95.75) (end 196.05625 94.44375) (width 0.25) (layer B.Cu) (net 12))
+  (segment (start 194.75 95.75) (end 215 95.75) (width 0.25) (layer F.Cu) (net 12))
+  (segment (start 215 95.75) (end 217 93.75) (width 0.25) (layer F.Cu) (net 12))
+  (via (at 217 93.75) (size 0.8) (drill 0.4) (layers F.Cu B.Cu) (net 12))
+  (segment (start 215.95625 88.16875) (end 215.10625 88.16875) (width 0.25) (layer B.Cu) (net 12))
+  (segment (start 217 89.2125) (end 215.95625 88.16875) (width 0.25) (layer B.Cu) (net 12))
+  (segment (start 217 93.75) (end 217 89.2125) (width 0.25) (layer B.Cu) (net 12))
+  (segment (start 217 93.75) (end 222 93.75) (width 0.25) (layer F.Cu) (net 12))
+  (segment (start 222 93.75) (end 223.75 95.5) (width 0.25) (layer F.Cu) (net 12))
+  (via (at 233 95.5) (size 0.8) (drill 0.4) (layers F.Cu B.Cu) (net 12))
+  (segment (start 223.75 95.5) (end 233 95.5) (width 0.25) (layer F.Cu) (net 12))
+  (segment (start 234.15625 94.34375) (end 234.15625 88.16875) (width 0.25) (layer B.Cu) (net 12))
+  (segment (start 233 95.5) (end 234.15625 94.34375) (width 0.25) (layer B.Cu) (net 12))
+  (via (at 251.75 95.5) (size 0.8) (drill 0.4) (layers F.Cu B.Cu) (net 12))
+  (segment (start 233 95.5) (end 251.75 95.5) (width 0.25) (layer F.Cu) (net 12))
+  (segment (start 253.20625 94.04375) (end 253.20625 88.16875) (width 0.25) (layer B.Cu) (net 12))
+  (segment (start 251.75 95.5) (end 253.20625 94.04375) (width 0.25) (layer B.Cu) (net 12))
+  (via (at 278 95.5) (size 0.8) (drill 0.4) (layers F.Cu B.Cu) (net 12))
+  (segment (start 251.75 95.5) (end 278 95.5) (width 0.25) (layer F.Cu) (net 12))
+  (segment (start 279.4 94.1) (end 279.4 88.16875) (width 0.25) (layer B.Cu) (net 12))
+  (segment (start 278 95.5) (end 279.4 94.1) (width 0.25) (layer B.Cu) (net 12))
+  (via (at 304.25 95.5) (size 0.8) (drill 0.4) (layers F.Cu B.Cu) (net 12))
+  (segment (start 278 95.5) (end 304.25 95.5) (width 0.25) (layer F.Cu) (net 12))
+  (segment (start 305.59375 94.15625) (end 305.59375 88.16875) (width 0.25) (layer B.Cu) (net 12))
+  (segment (start 304.25 95.5) (end 305.59375 94.15625) (width 0.25) (layer B.Cu) (net 12))
+  (via (at 321 95.5) (size 0.8) (drill 0.4) (layers F.Cu B.Cu) (net 12))
+  (segment (start 304.25 95.5) (end 321 95.5) (width 0.25) (layer F.Cu) (net 12))
+  (segment (start 322.2625 94.2375) (end 322.2625 88.9625) (width 0.25) (layer B.Cu) (net 12))
+  (segment (start 321 95.5) (end 322.2625 94.2375) (width 0.25) (layer B.Cu) (net 12))
   (segment (start 105.56875 46.8625) (end 105.56875 47.5625) (width 0.25) (layer B.Cu) (net 28))
   (segment (start 103.41875 44.7125) (end 105.56875 46.8625) (width 0.25) (layer B.Cu) (net 28))
