File: pcb/matrix.sch (KiCad schematic (older format))
At the start: 134 parts, among them K1 K_GRV, K10 K_LAPP, K11 K_2, K12 K_W, K13 K_S, K14 K_X, K15 K_LALT, K16 K_3, K17 K_E, K18 K_D, K19 K_C, K2 K_TAB, K20 K_4, K21 K_R, K22 K_F, K23 K_V, K24 K_5, K25 K_T, K26 K_G, K27 K_B, K28 K_SPC, K29 K_6, K3 K_CAPS_LOCK, K30 K_Y, K31 K_H, K32 K_N, K33 K_7, K34 K_U, K35 K_J, K36 K_M, K37 K_8, K38 K_I, K39 K_K, K4 K_LSHIFT, K40 K_COMMA, K41 K_9, K42 K_O, K43 K_L, K44 K_DOT, K45 K_0, K46 K_P, K47 K_SEMIC, K48 K_SLASH, K49 K_RALT, K5 K_LCTRL, K50 K_MINUS, K51 K_LBRC, K52 K_QUOTE, K53 K_RAPP, K54 K_EQUAL, K55 K_RBRC, K56 K_ENTER, K57 K_RSHIFT, K58 K_LEFT, K59 K_BACKSPACE, K6 K_1, K60 K_BSLSH, K61 K_UP, K62 K_DOWN, K63 K_PAGE_UP, K64 K_PAGE_DN, K65 K_INSERT, K66 K_DELETE, K67 K_RIGHT, K7 K_Q, K8 K_A, K9 K_Z

Commit message: routed switches vertical & diodes
Connections:
- net col11: now also K53.1
Changed lines of the file:
@@
 	6650 6400 11650 6400
 Connection ~ 6650 6400
+Wire Wire Line
+	13300 6000 13300 4000
+Connection ~ 13300 4000
 $EndSCHEMATC

Commit message: re-annotated everything in line instead of column
which is more clear for the matrix
Parts:
- renumbered D41 to D10, D45 to D11, D50 to D12, D54 to D13, D59 to D14, D63 to D15, D2 to D16, D7 to D17, D12 to D18, D17 to D19, D6 to D2, D21 to D20, D25 to D21, D30 to D22, D34 to D23, D38 to D24, D42 to D25, D46 to D26, D51 to D27, D55 to D28, D60 to D29, D11 to D3, D64 to D30, D3 to D31, D8 to D32, D13 to D33, D18 to D34, D22 to D35, D26 to D36, D31 to D37, D35 to D38, D16 to D4, D43 to D40, D47 to D41, D52 to D42, D56 to D43, D65 to D44, D4 to D45, D9 to D46, D14 to D47, D19 to D48, D23 to D49, D20 to D5, D27 to D50, D32 to D51, D36 to D52, D40 to D53, D44 to D54, D48 to D55, D57 to D56, D61 to D57, D66 to D58, D5 to D59, D24 to D6, D10 to D60, D15 to D61, D28 to D62, D49 to D63, D53 to D64, D58 to D65, D62 to D66, D29 to D7, D33 to D8, D37 to D9, K41 to K10, K45 to K11, K50 to K12, K54 to K13, K59 to K14, K63 to K15, K2 to K16, K7 to K17, K12 to K18, K17 to K19, K6 to K2, K21 to K20, K25 to K21, K30 to K22, K34 to K23, K38 to K24, K42 to K25, K46 to K26, K51 to K27, K55 to K28, K60 to K29, K11 to K3, K64 to K30, K3 to K31, K8 to K32, K13 to K33, K18 to K34, K22 to K35, K26 to K36, K31 to K37, K35 to K38, K16 to K4, K43 to K40, K47 to K41, K52 to K42, K56 to K43, K65 to K44, K4 to K45, K9 to K46, K14 to K47, K19 to K48, K23 to K49, K20 to K5, K27 to K50, K32 to K51, K36 to K52, K40 to K53, K44 to K54, K48 to K55, K57 to K56, K61 to K57, K66 to K58, K5 to K59, K24 to K6, K10 to K60, K15 to K61, K28 to K62, K49 to K63, K53 to K64, K58 to K65, K62 to K66, K29 to K7, K33 to K8, K37 to K9

Commit message: fix footprint of backslash
Parts:
- K29: footprint Alps_Only:ALPS-1U -> Alps_Only:ALPS-1.5U
Changed lines of the file:
@@
 F 0 "K29" H 15000 3233 60  0000 C CNN
 F 1 "K_BSLSH" H 15000 2900 60  0000 C CNN
-F 2 "Alps_Only:ALPS-1U" H 15000 3000 60  0001 C CNN
+F 2 "Alps_Only:ALPS-1.5U" H 15000 3000 60  0001 C CNN
 F 3 "" H 15000 3000 60  0000 C CNN
 	1    15000 3000

Commit message: renamed key values for silks layer
Parts:
- K1: value K_GRV -> GRV
- K10: value K_9 -> #9
- K11: value K_0 -> #0
- K12: value K_MINUS -> -_
- K13: value K_EQUAL -> =+
- K14: value K_BACKSPACE -> BACK
- K15: value K_PAGE_UP -> PAGE UP
- K16: value K_TAB -> TAB
- K17: value K_Q -> Q
- K18: value K_W -> E
- K19: value K_E -> E
- K2: value K_1 -> #1
- K20: value K_R -> R
- K21: value K_T -> T
- K22: value K_Y -> Y
- K23: value K_U -> U
- K24: value K_I -> I
- K25: value K_O -> O
- K26: value K_P -> P
- K27: value K_LBRC -> {[
- K28: value K_RBRC -> ]}
- K29: value K_BSLSH -> \\|
- K3: value K_2 -> #2
- K30: value K_PAGE_DN -> PAGE DN
- K31: value K_CAPS_LOCK -> CAPSLOCK
- K32: value K_A -> A
- K33: value K_S -> S
- K34: value K_D -> D
- K35: value K_F -> F
- K36: value K_G -> G
- K37: value K_H -> H
- K38: value K_J -> J
- K39: value K_K -> K
- K4: value K_3 -> #3
- K40: value K_L -> L
- K41: value K_SEMIC -> ;:
- K42: value K_QUOTE -> '\"
- K43: value K_ENTER -> ENTER
- K44: value K_INSERT -> INSERT
- K45: value K_LSHIFT -> LSHIFT
- K46: value K_Z -> Z
- K47: value K_X -> X
- K48: value K_C -> C
- K49: value K_V -> V
- K5: value K_4 -> #4
- K50: value K_B -> B
- K51: value K_N -> N
- K52: value K_M -> M
- K53: value K_COMMA -> ,<
- K54: value K_DOT -> .>
- K55: value K_SLASH -> /?
- K56: value K_RSHIFT -> RSHIFT
- K57: value K_UP -> UP
- K58: value K_DELETE -> DEL
- K59: value K_LCTRL -> LCTRL
- K6: value K_5 -> #5
- K60: value K_LAPP -> LALT
- K61: value K_LALT -> LCOMMAND
- K62: value K_SPC -> SPACE
- K63: value K_RALT -> RCOMMAND
- K64: value K_RAPP -> RALT
- K65: value K_LEFT -> LEFT
- K66: value K_DOWN -> DOWN
- K67: value K_RIGHT -> RIGHT
- K7: value K_6 -> #6
- K8: value K_7 -> #7
- K9: value K_8 -> #8
